Commit message: add precision_landing

File: sitl_config/ugv/catvehicle/urdf/catvehicle1-3.xacro (robot description, xacro)
@@ -583,5 +583,5 @@
               <origin xyz="0 -0.5 0.05" rpy="0 1.57 1.57"/>
               <geometry>
-                <mesh filename="model://qrcode1-3/meshes/qrcode1-3.dae" scale="2 5 2"/>
+                <mesh filename="model://apriltag0-2/meshes/apriltag0-2.dae" scale="2 5 2"/>
               </geometry>
             </visual>
