Commit message: update

File: sitl_config/ugv/catvehicle/urdf/catvehicle.urdf (robot description, URDF)
Before this commit: robot catvehicle, 14 links, 13 joints
Links:
- removed link parking_link
- added link camera_link, mass 1e-5; collision box size=0.25 0.25 0.25; visual box size=0.25 0.25 0.25
Joints:
- removed joint parking_joint
- added joint camera_joint: type fixed, parent base_link, child camera_link, origin xyz=0 0 2.1 rpy=0 0 0, axis 0 0 1
