Commit message: modify robotic arm

File: sitl_config/robotic_arm/le_arm/urdf/component_snippets.xacro (robot description, xacro)
@@ -556,5 +556,5 @@
         <noiseUniformAngularVelocity>${noise_uniform_angular_velocity}</noiseUniformAngularVelocity>  <!-- symmetric bounds of uniform noise [rad/s] -->
         <xacro:if value="${enable_odometry_map}">
-          <covarianceImage>file:///home/robin/le_arm_ws/src/rotors_gazebo/resource/${odometry_map}</covarianceImage>
+          <covarianceImage>package://rotors_gazebo/resource/${odometry_map}</covarianceImage>
           <covarianceImageScale>${image_scale}</covarianceImageScale>
         </xacro:if>

File: sitl_config/robotic_arm/le_arm/urdf/le_arm.urdf.xacro (robot description, xacro)
@@ -24,19 +24,19 @@
             <geometry>
                 <mesh
-                filename="file:///home/robin/le_arm_ws/src/le_arm/meshes/arm/base_link.STL" />
-            </geometry>
-            <material
-                name="">
-                <color
-                rgba="0.75294 0.75294 0.75294 1" />
-            </material>
-            </visual>
-            <collision>
-            <origin
-                xyz="0 0 0"
-                rpy="0 0 0" />
-            <geometry>
-                <mesh
-                filename="file:///home/robin/le_arm_ws/src/le_arm/meshes/arm/base_link.STL" />
+                filename="package://le_arm/meshes/arm/base_link.STL" />
+            </geometry>
+            <material
+                name="">
+                <color
+                rgba="0.75294 0.75294 0.75294 1" />
+            </material>
+            </visual>
+            <collision>
+            <origin
+                xyz="0 0 0"
+                rpy="0 0 0" />
+            <geometry>
+                <mesh
+                filename="package://le_arm/meshes/arm/base_link.STL" />
             </geometry>
             </collision>
@@ -64,19 +64,19 @@
             <geometry>
                 <mesh
-                filename="file:///home/robin/le_arm_ws/src/le_arm/meshes/arm/shoulder_link.STL" />
-            </geometry>
-            <material
-                name="">
-                <color
-                rgba="0.75294 0.75294 0.75294 1" />
-            </material>
-            </visual>
-            <collision>
-            <origin
-                xyz="0 0 0"
-                rpy="0 0 0" />
-            <geometry>
-                <mesh
-                filename="file:///home/robin/le_arm_ws/src/le_arm/meshes/arm/shoulder_link.STL" />
+                filename="package://le_arm/meshes/arm/shoulder_link.STL" />
+            </geometry>
+            <material
+                name="">
+                <color
+                rgba="0.75294 0.75294 0.75294 1" />
+            </material>
+            </visual>
+            <collision>
+            <origin
+                xyz="0 0 0"
+                rpy="0 0 0" />
+            <geometry>
+                <mesh
+                filename="package://le_arm/meshes/arm/shoulder_link.STL" />
             </geometry>
             </collision>
@@ -122,19 +122,19 @@
             <geometry>
                 <mesh
-                filename="file:///home/robin/le_arm_ws/src/le_arm/meshes/arm/upper_arm_link.STL" />
-            </geometry>
-            <material
-                name="">
-                <color
-                rgba="0.75294 0.75294 0.75294 1" />
-            </material>
-            </visual>
-            <collision>
-            <origin
-                xyz="0 0 0"
-                rpy="0 0 0" />
-            <geometry>
-                <mesh
-                filename="file:///home/robin/le_arm_ws/src/le_arm/meshes/arm/upper_arm_link.STL" />
+                filename="package://le_arm/meshes/arm/upper_arm_link.STL" />
+            </geometry>
+            <material
+                name="">
+                <color
+                rgba="0.75294 0.75294 0.75294 1" />
+            </material>
+            </visual>
+            <collision>
+            <origin
+                xyz="0 0 0"
+                rpy="0 0 0" />
+            <geometry>
+                <mesh
+                filename="package://le_arm/meshes/arm/upper_arm_link.STL" />
             </geometry>
             </collision>
@@ -180,19 +180,19 @@
             <geometry>
                 <mesh
-                filename="file:///home/robin/le_arm_ws/src/le_arm/meshes/arm/forearm_link.STL" />
-            </geometry>
-            <material
-                name="">
-                <color
-                rgba="0.75294 0.75294 0.75294 1" />
-            </material>
-            </visual>
-            <collision>
-            <origin
-                xyz="0 0 0"
-                rpy="0 0 0" />
-            <geometry>
-                <mesh
-                filename="file:///home/robin/le_arm_ws/src/le_arm/meshes/arm/forearm_link.STL" />
+                filename="package://le_arm/meshes/arm/forearm_link.STL" />
+            </geometry>
+            <material
+                name="">
+                <color
+                rgba="0.75294 0.75294 0.75294 1" />
+            </material>
+            </visual>
+            <collision>
+            <origin
+                xyz="0 0 0"
+                rpy="0 0 0" />
+            <geometry>
+                <mesh
+                filename="package://le_arm/meshes/arm/forearm_link.STL" />
             </geometry>
             </collision>
@@ -238,19 +238,19 @@
             <geometry>
                 <mesh
-                filename="file:///home/robin/le_arm_ws/src/le_arm/meshes/arm/wrist_1_link.STL" />
-            </geometry>
-            <material
-                name="">
-                <color
-                rgba="0.75294 0.75294 0.75294 1" />
-            </material>
-            </visual>
-            <collision>
-            <origin
-                xyz="0 0 0"
-                rpy="0 0 0" />
-            <geometry>
-                <mesh
-                filename="file:///home/robin/le_arm_ws/src/le_arm/meshes/arm/wrist_1_link.STL" />
+                filename="package://le_arm/meshes/arm/wrist_1_link.STL" />
+            </geometry>
+            <material
+                name="">
+                <color
+                rgba="0.75294 0.75294 0.75294 1" />
+            </material>
+            </visual>
+            <collision>
+            <origin
+                xyz="0 0 0"
+                rpy="0 0 0" />
+            <geometry>
+                <mesh
+                filename="package://le_arm/meshes/arm/wrist_1_link.STL" />
             </geometry>
             </collision>

File: sitl_config/robotic_arm/le_arm/urdf/le_arm_gripper.urdf.xacro (robot description, xacro)
@@ -25,19 +25,19 @@
             <geometry>
                 <mesh
-                filename="file:///home/robin/le_arm_ws/src/le_arm/meshes/gripper/base_link.STL" />
-            </geometry>
-            <material
-                name="">
-                <color
-                rgba="0.75294 0.75294 0.75294 1" />
-            </material>
-            </visual>
-            <collision>
-            <origin
-                xyz="0 0 0"
-                rpy="0 0 0" />
-            <geometry>
-                <mesh
-                filename="file:///home/robin/le_arm_ws/src/le_arm/meshes/gripper/base_link.STL" />
+                filename="package://le_arm/meshes/gripper/base_link.STL" />
+            </geometry>
+            <material
+                name="">
+                <color
+                rgba="0.75294 0.75294 0.75294 1" />
+            </material>
+            </visual>
+            <collision>
+            <origin
+                xyz="0 0 0"
+                rpy="0 0 0" />
+            <geometry>
+                <mesh
+                filename="package://le_arm/meshes/gripper/base_link.STL" />
             </geometry>
             </collision>
@@ -65,19 +65,19 @@
             <geometry>
                 <mesh
-                filename="file:///home/robin/le_arm_ws/src/le_arm/meshes/gripper/left_knuckle_link.STL" />
-            </geometry>
-            <material
-                name="">
-                <color
-                rgba="0.75294 0.75294 0.75294 1" />
-            </material>
-            </visual>
-            <collision>
-            <origin
-                xyz="0 0 0"
-                rpy="0 0 0" />
-            <geometry>
-                <mesh
-                filename="file:///home/robin/le_arm_ws/src/le_arm/meshes/gripper/left_knuckle_link.STL" />
+                filename="package://le_arm/meshes/gripper/left_knuckle_link.STL" />
+            </geometry>
+            <material
+                name="">
+                <color
+                rgba="0.75294 0.75294 0.75294 1" />
+            </material>
+            </visual>
+            <collision>
+            <origin
+                xyz="0 0 0"
+                rpy="0 0 0" />
+            <geometry>
+                <mesh
+                filename="package://le_arm/meshes/gripper/left_knuckle_link.STL" />
             </geometry>
             </collision>
@@ -123,19 +123,19 @@
             <geometry>
                 <mesh
-                filename="file:///home/robin/le_arm_ws/src/le_arm/meshes/gripper/right_knuckle_link.STL" />
-            </geometry>
-            <material
-                name="">
-                <color
-                rgba="0.75294 0.75294 0.75294 1" />
-            </material>
-            </visual>
-            <collision>
-            <origin
-                xyz="0 0 0"
-                rpy="0 0 0" />
-            <geometry>
-                <mesh
-                filename="file:///home/robin/le_arm_ws/src/le_arm/meshes/gripper/right_knuckle_link.STL" />
+                filename="package://le_arm/meshes/gripper/right_knuckle_link.STL" />
+            </geometry>
+            <material
+                name="">
+                <color
+                rgba="0.75294 0.75294 0.75294 1" />
+            </material>
+            </visual>
+            <collision>
+            <origin
+                xyz="0 0 0"
+                rpy="0 0 0" />
+            <geometry>
+                <mesh
+                filename="package://le_arm/meshes/gripper/right_knuckle_link.STL" />
             </geometry>
             </collision>
@@ -182,19 +182,19 @@
             <geometry>
                 <mesh
-                filename="file:///home/robin/le_arm_ws/src/le_arm/meshes/gripper/left_inner_knuckle_link.STL" />
-            </geometry>
-            <material
-                name="">
-                <color
-                rgba="0.75294 0.75294 0.75294 1" />
-            </material>
-            </visual>
-            <collision>
-            <origin
-                xyz="0 0 0"
-                rpy="0 0 0" />
-            <geometry>
-                <mesh
-                filename="file:///home/robin/le_arm_ws/src/le_arm/meshes/gripper/left_inner_knuckle_link.STL" />
+                filename="package://le_arm/meshes/gripper/left_inner_knuckle_link.STL" />
+            </geometry>
+            <material
+                name="">
+                <color
+                rgba="0.75294 0.75294 0.75294 1" />
+            </material>
+            </visual>
+            <collision>
+            <origin
+                xyz="0 0 0"
+                rpy="0 0 0" />
+            <geometry>
+                <mesh
+                filename="package://le_arm/meshes/gripper/left_inner_knuckle_link.STL" />
             </geometry>
             </collision>
@@ -241,19 +241,19 @@
             <geometry>
                 <mesh
-                filename="file:///home/robin/le_arm_ws/src/le_arm/meshes/gripper/left_finger_link.STL" />
-            </geometry>
-            <material
-                name="">
-                <color
-                rgba="0.75294 0.75294 0.75294 1" />
-            </material>
-            </visual>
-            <collision>
-            <origin
-                xyz="0 0 0"
-                rpy="0 0 0" />
-            <geometry>
-                <mesh
-                filename="file:///home/robin/le_arm_ws/src/le_arm/meshes/gripper/left_finger_link.STL" />
+                filename="package://le_arm/meshes/gripper/left_finger_link.STL" />
+            </geometry>
+            <material
+                name="">
+                <color
+                rgba="0.75294 0.75294 0.75294 1" />
+            </material>
+            </visual>
+            <collision>
+            <origin
+                xyz="0 0 0"
+                rpy="0 0 0" />
+            <geometry>
+                <mesh
+                filename="package://le_arm/meshes/gripper/left_finger_link.STL" />
             </geometry>
             </collision>
@@ -300,19 +300,19 @@
             <geometry>
                 <mesh
-                filename="file:///home/robin/le_arm_ws/src/le_arm/meshes/gripper/right_inner_knuckle_link.STL" />
-            </geometry>
-            <material
-                name="">
-                <color
-                rgba="0.75294 0.75294 0.75294 1" />
-            </material>
-            </visual>
-            <collision>
-            <origin
-                xyz="0 0 0"
-                rpy="0 0 0" />
-            <geometry>
-                <mesh
-                filename="file:///home/robin/le_arm_ws/src/le_arm/meshes/gripper/right_inner_knuckle_link.STL" />
+                filename="package://le_arm/meshes/gripper/right_inner_knuckle_link.STL" />
+            </geometry>
+            <material
+                name="">
+                <color
+                rgba="0.75294 0.75294 0.75294 1" />
+            </material>
+            </visual>
+            <collision>
+            <origin
+                xyz="0 0 0"
+                rpy="0 0 0" />
+            <geometry>
+                <mesh
+                filename="package://le_arm/meshes/gripper/right_inner_knuckle_link.STL" />
             </geometry>
             </collision>
@@ -359,19 +359,19 @@
             <geometry>
                 <mesh
-                filename="file:///home/robin/le_arm_ws/src/le_arm/meshes/gripper/right_finger_link.STL" />
-            </geometry>
-            <material
-                name="">
-                <color
-                rgba="0.75294 0.75294 0.75294 1" />
-            </material>
-            </visual>
-            <collision>
-            <origin
-                xyz="0 0 0"
-                rpy="0 0 0" />
-            <geometry>
-                <mesh
-                filename="file:///home/robin/le_arm_ws/src/le_arm/meshes/gripper/right_finger_link.STL" />
+                filename="package://le_arm/meshes/gripper/right_finger_link.STL" />
+            </geometry>
+            <material
+                name="">
+                <color
+                rgba="0.75294 0.75294 0.75294 1" />
+            </material>
+            </visual>
+            <collision>
+            <origin
+                xyz="0 0 0"
+                rpy="0 0 0" />
+            <geometry>
+                <mesh
+                filename="package://le_arm/meshes/gripper/right_finger_link.STL" />
             </geometry>
             </collision>

File: sitl_config/robotic_arm/le_arm/urdf/multirotor_base.xacro (robot description, xacro)
@@ -85,5 +85,5 @@
         <origin xyz="0 0 0" rpy="0 0 0" />
         <geometry>
-          <mesh filename="file:///home/robin/le_arm_ws/src/le_arm/meshes/iris/${mesh_file}"
+          <mesh filename="package://le_arm/meshes/iris/${mesh_file}"
             scale="${mesh_scale}" />
           <!-- <box size="${body_width} ${body_width} ${body_height}"/> --> <!-- [m] [m] [m] -->
@@ -144,6 +144,6 @@
         <geometry>
           <!-- <cylinder length="0.005" radius="${radius_rotor}"/> --> <!-- [m] -->
-          <!-- <mesh filename="file:///home/robin/le_arm_ws/src/le_arm/meshes/propeller_${direction}.dae" -->
-          <mesh filename="file:///home/robin/le_arm_ws/src/le_arm/meshes/iris/${mesh}_${direction}.dae"
+          <!-- <mesh filename="package://le_arm/meshes/propeller_${direction}.dae" -->
+          <mesh filename="package://le_arm/meshes/iris/${mesh}_${direction}.dae"
             scale="${mesh_scale}" />
           <!-- <box size="${2*radius_rotor} 0.01 0.005"/> -->

File: sitl_config/robotic_arm/le_arm/urdf/sensors/camera.urdf.xacro (robot description, xacro)
@@ -14,5 +14,5 @@
            <origin xyz="0 0 0" rpy="0 0 0"/>
            <geometry>
-           <mesh filename="file:///home/robin/le_arm_ws/src/le_arm/meshes/sensors/camera.STL" />
+           <mesh filename="package://le_arm/meshes/sensors/camera.STL" />
            </geometry>
        </collision>
@@ -20,5 +20,5 @@
            <origin xyz="0 0 0" rpy="-3.14 0 -1.57"/>
            <geometry>
-           <mesh filename="file:///home/robin/le_arm_ws/src/le_arm/meshes/sensors/camera.STL" />
+           <mesh filename="package://le_arm/meshes/sensors/camera.STL" />
            </geometry>
            <material name="red"/>

Commit message: modify for robotic arm

File: sitl_config/robotic_arm/le_arm/urdf/component_snippets.xacro (robot description, xacro)
@@ -679,7 +679,5 @@
         <origin xyz="0 0 0" rpy="0 0 0" />
         <geometry>
-         <box>
-            <size>0.015 0.1 0.02</size>
-          </box>
+         <box size="0.015 0.1 0.02" />
         </geometry>
       </collision>
@@ -687,7 +685,5 @@
         <origin xyz="0 0 0" rpy="0 0 0" />
         <geometry>
-          <box>
-            <size>0.015 0.1 0.02</size>
-          </box>
+          <box size="0.015 0.1 0.02" />
         </geometry>
       </visual>

File: sitl_config/robotic_arm/le_arm/urdf/iris_arm_base.xacro (robot description, xacro)
@@ -188,6 +188,7 @@
   </xacro:if>
   <!-- Instantiate a VI sensor. -->
-  <xacro:vi_sensor_macro namespace="$(arg name)" parent_link="base_link">
+  <!-- <xacro:vi_sensor_macro namespace="$(arg name)" parent_link="base_link">
   <origin xyz="0.2 0.0 0.0" rpy="0.0 0.0 0.0" />
-  </xacro:vi_sensor_macro>
+  </xacro:vi_sensor_macro> -->
+  <xacro:include filename="$(find le_arm)/urdf/sensors/camera.urdf.xacro"/>
 </robot>

File: sitl_config/robotic_arm/le_arm/urdf/sensors/camera.urdf.xacro (robot description, xacro)
@@ -5,5 +5,5 @@
 <robot name="camera" xmlns:xacro="http://ros.org/wiki/xacro">
    <joint name="camera_joint" type="fixed">
-        <origin xyz="0.3 0 0.7" rpy="0 1.57 0"/>
+        <origin xyz="0.05 0 -0.07" rpy="0 1.57 0"/>
         <parent link="base_link"/>
         <child link="camera_link"/>
@@ -14,5 +14,5 @@
            <origin xyz="0 0 0" rpy="0 0 0"/>
            <geometry>
-           <mesh filename="package://le_arm/meshes/sensors/camera.STL" />
+            <mesh filename="package://le_arm/meshes/sensors/camera.STL" scale="0.1 0.1 0.1" />
            </geometry>
        </collision>
@@ -27,7 +27,7 @@
         <mass value="0.00001" />
         <origin xyz="0 0 0" />
-        <inertia ixx="0.001" ixy="0.0" ixz="0.0"
-          iyy="0.001" iyz="0.0"
-          izz="0.001" />
+        <inertia ixx="0.00001" ixy="0.0" ixz="0.0"
+          iyy="0.00001" iyz="0.0"
+          izz="0.00001" />
        </inertial>
    </link>
